File: Equemetico.sch (EAGLE design)
At the start: 18 parts, among them IC1 RASPBERRY_PI_ZERO_W_(V1.3), K1 SRD-05VDC-SL-C, K2 SRD-05VDC-SL-C, K3 SRD-05VDC-SL-C, K4 SRD-05VDC-SL-C, K5 SRD-05VDC-SL-C

Commit message: movi el pir
movi  el pir
Parts:
- added OK1, OK2: TLP283-4, optocoupler:TLP283-4
- added OK4: TLP283, optocoupler:TLP283
Connections:
- new net N$11: K1.4
- new net N$12: X1-2.1
- new net N$13: K2.4
Other:
- moved on the sheet: U$1, X2-1, X2-2
Changed lines of the file:
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@@
 <setting verticaltext="up"/>
 </settings>
-<grid distance="0.1" unitdist="inch" unit="inch" style="lines" multiple="1" display="yes" altdistance="0.01" altunitdist="inch" altunit="inch"/>
+<grid distance="0.1" unitdist="inch" unit="inch" style="lines" multiple="1" display="no" altdistance="0.01" altunitdist="inch" altunit="inch"/>
 <layers>
 <layer number="1" name="Top" color="4" fill="1" visible="no" active="no"/>
@@
 <part name="D4" library="diode" library_urn="urn:adsk.eagle:library:210" deviceset="1N4004" device="" package3d_urn="urn:adsk.eagle:package:43336/1"/>
 <part name="D5" library="diode" library_urn="urn:adsk.eagle:library:210" deviceset="1N4004" device="" package3d_urn="urn:adsk.eagle:package:43336/1"/>
+<part name="OK1" library="optocoupler" library_urn="urn:adsk.eagle:library:320" deviceset="TLP283-4" device="" package3d_urn="urn:adsk.eagle:package:21967/1"/>
+<part name="OK2" library="optocoupler" library_urn="urn:adsk.eagle:library:320" deviceset="TLP283-4" device="" package3d_urn="urn:adsk.eagle:package:21967/1"/>
+<part name="OK4" library="optocoupler" library_urn="urn:adsk.eagle:library:320" deviceset="TLP283" device="" package3d_urn="urn:adsk.eagle:package:21958/1"/>
 </parts>
 <sheets>
@@
 <attribute name="VALUE" x="107.95" y="241.3" size="1.778" layer="96" align="center-left"/>
 </instance>
-<instance part="U$1" gate="G$1" x="170.18" y="210.82" smashed="yes">
-<attribute name="NAME" x="157.48" y="231.14" size="1.778" layer="95"/>
-<attribute name="VALUE" x="157.48" y="228.6" size="1.778" layer="96"/>
+<instance part="U$1" gate="G$1" x="152.4" y="208.28" smashed="yes">
+<attribute name="NAME" x="139.7" y="228.6" size="1.778" layer="95"/>
+<attribute name="VALUE" x="139.7" y="226.06" size="1.778" layer="96"/>
 </instance>
 <instance part="K1" gate="G$1" x="-10.16" y="281.94" smashed="yes">
@@
 <attribute name="VALUE" x="16.764" y="273.558" size="1.778" layer="96"/>
 </instance>
-<instance part="X2" gate="-1" x="68.58" y="281.94" smashed="yes">
-<attribute name="NAME" x="72.136" y="281.305" size="1.778" layer="95"/>
-</instance>
-<instance part="X2" gate="-2" x="68.58" y="276.86" smashed="yes">
-<attribute name="NAME" x="72.136" y="276.225" size="1.778" layer="95"/>
-<attribute name="VALUE" x="67.564" y="273.558" size="1.778" layer="96"/>
+<instance part="X2" gate="-1" x="73.66" y="281.94" smashed="yes">
+<attribute name="NAME" x="77.216" y="281.305" size="1.778" layer="95"/>
+</instance>
+<instance part="X2" gate="-2" x="73.66" y="276.86" smashed="yes">
+<attribute name="NAME" x="77.216" y="276.225" size="1.778" layer="95"/>
+<attribute name="VALUE" x="72.644" y="273.558" size="1.778" layer="96"/>
 </instance>
 <instance part="X3" gate="-1" x="119.38" y="281.94" smashed="yes">
@@
 <attribute name="NAME" x="192.5574" y="287.02" size="1.778" layer="95" rot="R90"/>
 <attribute name="VALUE" x="195.3514" y="287.02" size="1.778" layer="96" rot="R90"/>
+</instance>
+<instance part="OK1" gate="A" x="-48.26" y="182.88" smashed="yes">
+<attribute name="NAME" x="-55.245" y="188.595" size="1.778" layer="95"/>
+<attribute name="VALUE" x="-55.245" y="175.26" size="1.778" layer="96"/>
+</instance>
+<instance part="OK1" gate="B" x="-25.4" y="182.88" smashed="yes">
+<attribute name="NAME" x="-32.385" y="188.595" size="1.778" layer="95"/>
+<attribute name="VALUE" x="-32.385" y="175.26" size="1.778" layer="96"/>
+</instance>
+<instance part="OK1" gate="C" x="-5.08" y="182.88" smashed="yes">
+<attribute name="NAME" x="-12.065" y="188.595" size="1.778" layer="95"/>
+<attribute name="VALUE" x="-12.065" y="175.26" size="1.778" layer="96"/>
+</instance>
+<instance part="OK1" gate="D" x="15.24" y="182.88" smashed="yes">
+<attribute name="NAME" x="8.255" y="188.595" size="1.778" layer="95"/>
+<attribute name="VALUE" x="8.255" y="175.26" size="1.778" layer="96"/>
+</instance>
+<instance part="OK2" gate="A" x="91.44" y="256.54" smashed="yes">
+<attribute name="NAME" x="84.455" y="262.255" size="1.778" layer="95"/>
+<attribute name="VALUE" x="84.455" y="248.92" size="1.778" layer="96"/>
+</instance>
+<instance part="OK2" gate="B" x="114.3" y="256.54" smashed="yes">
+<attribute name="NAME" x="107.315" y="262.255" size="1.778" layer="95"/>
+<attribute name="VALUE" x="107.315" y="248.92" size="1.778" layer="96"/>
+</instance>
+<instance part="OK2" gate="C" x="144.78" y="256.54" smashed="yes">
+<attribute name="NAME" x="137.795" y="262.255" size="1.778" layer="95"/>
+<attribute name="VALUE" x="137.795" y="248.92" size="1.778" layer="96"/>
+</instance>
+<instance part="OK2" gate="D" x="167.64" y="256.54" smashed="yes">
+<attribute name="NAME" x="160.655" y="262.255" size="1.778" layer="95"/>
+<attribute name="VALUE" x="160.655" y="248.92" size="1.778" layer="96"/>
+</instance>
+<instance part="OK4" gate="G$1" x="193.04" y="256.54" smashed="yes">
+<attribute name="NAME" x="186.055" y="262.255" size="1.778" layer="95"/>
+<attribute name="VALUE" x="186.055" y="248.92" size="1.778" layer="96"/>
 </instance>
 </instances>
@@
 <segment>
 <pinref part="X2" gate="-1" pin="1"/>
-<wire x1="66.04" y1="281.94" x2="66.04" y2="287.02" width="0.1524" layer="91"/>
-<label x="66.04" y="281.94" size="1.778" layer="95" rot="R90"/>
+<wire x1="71.12" y1="281.94" x2="71.12" y2="287.02" width="0.1524" layer="91"/>
+<label x="71.12" y="281.94" size="1.778" layer="95" rot="R90"/>
 </segment>
 </net>
@@
 </segment>
 </net>
+<net name="N$11" class="0">
+<segment>
+<pinref part="K1" gate="G$1" pin="4"/>
+<wire x1="5.08" y1="294.64" x2="5.08" y2="299.72" width="0.1524" layer="91"/>
+</segment>
+</net>
+<net name="N$12" class="0">
+<segment>
+<pinref part="X1" gate="-2" pin="1"/>
+<wire x1="15.24" y1="276.86" x2="12.7" y2="276.86" width="0.1524" layer="91"/>
+<wire x1="12.7" y1="276.86" x2="12.7" y2="269.24" width="0.1524" layer="91"/>
+</segment>
+</net>
+<net name="N$13" class="0">
+<segment>
+<pinref part="K2" gate="G$1" pin="4"/>
+<wire x1="60.96" y1="294.64" x2="60.96" y2="299.72" width="0.1524" layer="91"/>
+</segment>
+</net>

Commit message: Coenexion de relevadores
Relevadores conectados
Parts:
- added R1, R2, R3, R4, R5, R6, R7, R8, R9: (no value), rcl:R-US_R0402
Connections:
- removed net N$1: D1.C, K1.2
- removed net N$2: D1.A, K1.3
- removed net N$3: D2.C, K2.2
- removed net N$4: D2.A, K2.3
- removed net N$9: D5.C, K5.2
- new net 5V: D1.C, D2.C, D3.C, D4.C, D5.C, IC1.+5V_1, K1.2, K2.2, K3.2, K4.2, K5.2, PS1.+VO
- new net GND: IC1.GND_1, OK2A.EMIT, OK2B.EMIT, OK2C.EMIT, OK2D.EMIT, OK4.EMIT, PS1.-VO, R1.1, R2.1, R3.1, R4.1, R5.1
- new net INT1: IC1.GPIO_4/GPCLK0, OK2A.A
- new net INT2: IC1.GPIO27, OK2B.A
- new net INT3: IC1.GPIO_22, OK2C.A
- new net INT4: IC1.GPIO_23, OK2D.A
- new net INT5: IC1.GPIO_25, OK4.A
- new net N$14: OK4.C, R5.2
- new net N$30: D5.A, K5.3, OK4.COL
- new net N$32: D4.A, K4.3, OK2D.COL
- new net N$33: D3.A, K3.3, OK2C.COL
- new net N$34: D2.A, K2.3, OK2B.COL
- new net N$35: D1.A, K1.3, OK2A.COL
- new net NO1: K1.4, X1-2.1
- new net NO2: K2.4, X2-2.1
- new net NO3: K3.4, X3-2.1
- new net NO4: K4.4, X4-2.1
- new net NO5: K5.4, X5-2.1
- net N$10: now also OK2A.C, R1.2; no longer D5.A, K5.3
- net N$11: now also OK2B.C, R2.2; no longer K1.4
- net N$12: now also OK2C.C, R3.2; no longer X1-2.1
- net N$13: now also OK2D.C, R4.2; no longer K2.4
- net N$5: now also IC1.GPIO19/SPI0_MISO1/PWM1; no longer D3.C, K3.2
- net N$6: now also IC1.GPIO13/PWM1; no longer D3.A, K3.3
- net N$7: now also IC1.GPIO12/PWM0; no longer D4.C, K4.2
- net N$8: now also IC1.GPIO5//GPCLK1; no longer D4.A, K4.3
Other:
- moved on the sheet: D1, D2, D3, D4, D5, IC1, K1, K2, K3, K4, K5, OK1A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

Commit message: Conexion de las entradas
Entradas optoacopladas
Parts:
- added AC_INT, INT_1, INT_2, INT_3, INT_4: (no value), con-phoenix-254:MPT2
- added IC2: (no value), v-reg:XC63FPM
- added R10, R11, R12, R13: 1k, rcl:R-US_R0402
- R1, R2, R3, R4, R5, R6, R7, R8, R9: value (none) -> 220
Connections:
- removed net N$5: IC1.GPIO19/SPI0_MISO1/PWM1
- removed net N$6: IC1.GPIO13/PWM1
- removed net N$7: IC1.GPIO12/PWM0
- removed net N$8: IC1.GPIO5//GPCLK1
- new net 3.3V: IC2.OUT, R10.2, R11.2, R12.2, R13.2, U$1.VCC
- new net N$1: AC_INT-2.1, PS1.AC_1
- new net N$15: OK1B.C, R7.2
- new net N$16: INT_3-2.1, R8.2
- new net N$17: OK1C.C, R8.1
- new net N$18: INT_4-2.1, R9.2
- new net N$19: OK1D.C, R9.1
- new net N$2: AC_INT-1.1, PS1.AC_2
- new net N$3: INT_1-2.1, R6.1
- new net N$4: OK1A.C, R6.2
- new net N$9: INT_2-2.1, R7.1
- new net OUT1: IC1.GPIO_4/GPCLK0, OK2A.A
- new net OUT2: IC1.GPIO27, OK2B.A
- new net OUT3: IC1.GPIO_22, OK2C.A
- new net OUT4: IC1.GPIO_23, OK2D.A
- new net OUT5: IC1.GPIO_25, OK4.A
- net 5V: now also IC2.IN, OK1A.A, OK1B.A, OK1C.A, OK1D.A
- net GND: now also IC2.GND, INT_1-1.1, INT_2-1.1, INT_3-1.1, INT_4-1.1, OK1A.EMIT, OK1B.EMIT, OK1C.EMIT, OK1D.EMIT, U$1.GND
- net INT1: now also IC1.GPIO5//GPCLK1, OK1A.COL, R10.1; no longer IC1.GPIO_4/GPCLK0, OK2A.A
- net INT2: now also IC1.GPIO12/PWM0, OK1B.COL, R11.1; no longer IC1.GPIO27, OK2B.A
- net INT3: now also IC1.GPIO13/PWM1, OK1C.COL, R12.1; no longer IC1.GPIO_22, OK2C.A
- net INT4: now also IC1.GPIO19/SPI0_MISO1/PWM1, OK1D.COL, R13.1; no longer IC1.GPIO_23, OK2D.A
- net INT5: now also IC1.GPIO26, U$1.OUT; no longer IC1.GPIO_25, OK4.A
Other:
- moved on the sheet: IC1, OK1A, OK1B, OK1C, OK1D, PS1, R6, R7, R8, R9, U$1
