File: Diagramas/Esquematico/Esquematico.sch (EAGLE design)
At the start: 48 parts, among them IC1 RASPBERRY_PI_ZERO_W_(V1.3), IC2 3071, IC3 DS3231N_DIP, J1 Modulo Pir, K1 SRD-05VDC-SL-C, K2 SRD-05VDC-SL-C, K3 SRD-05VDC-SL-C, K4 SRD-05VDC-SL-C, U1 RFM69HW-868S2

Commit message: Ceacion del pcb
Parts:
- NEO_PIXEL: device con-wago-508:W232-3 -> con-wago-500:W237-102
Connections:
- net 5V: no longer NEO_PIXEL-2.SK
- net G18: now also NEO_PIXEL-1.KL; no longer NEO_PIXEL-1.SK
- net GND: now also NEO_PIXEL-2.KL; no longer NEO_PIXEL-3.SK
Changed lines of the file:
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@@
 <part name="R13" library="rcl" library_urn="urn:adsk.eagle:library:334" deviceset="R-US_" device="R0402" package3d_urn="urn:adsk.eagle:package:23547/3" value="1k"/>
 <part name="IC2" library="3071" deviceset="3071" device=""/>
-<part name="NEO_PIXEL" library="con-wago-508" library_urn="urn:adsk.eagle:library:196" deviceset="W232-3" device="" package3d_urn="urn:adsk.eagle:package:10743/1"/>
 <part name="BT1" library="CR2032_MFR_RH" deviceset="CR2032_MFR_RH" device=""/>
 <part name="IC3" library="DS3231N_DIP" deviceset="DS3231N_DIP" device=""/>
@@
 <part name="ANT1" library="RECE.20279.001E.01" deviceset="RECE.20279.001E.01" device=""/>
 <part name="C1" library="microbuilder" deviceset="CAP_CERAMIC" device="_0805" value="0.1F"/>
+<part name="NEO_PIXEL" library="con-wago-500" library_urn="urn:adsk.eagle:library:195" deviceset="W237-102" device="" package3d_urn="urn:adsk.eagle:package:10688/1"/>
 </parts>
 <sheets>
@@
 <attribute name="VALUE" x="-140.97" y="228.6" size="1.778" layer="96" align="center-left"/>
 </instance>
-<instance part="NEO_PIXEL" gate="-1" x="-99.06" y="226.06" smashed="yes">
-<attribute name="NAME" x="-105.918" y="226.949" size="1.778" layer="95" rot="R180"/>
-</instance>
-<instance part="NEO_PIXEL" gate="-2" x="-99.06" y="220.98" smashed="yes">
-<attribute name="NAME" x="-105.918" y="221.869" size="1.778" layer="95" rot="R180"/>
-</instance>
-<instance part="NEO_PIXEL" gate="-3" x="-99.06" y="215.9" smashed="yes">
-<attribute name="VALUE" x="-107.188" y="212.344" size="1.778" layer="96"/>
-<attribute name="NAME" x="-106.045" y="216.789" size="1.778" layer="95" rot="R180"/>
-</instance>
 <instance part="BT1" gate="G$1" x="-116.84" y="246.38" smashed="yes">
 <attribute name="NAME" x="-97.79" y="254" size="1.778" layer="95" align="center-left"/>
@@
 <attribute name="NAME" x="-53.34" y="271.78" size="1.27" layer="95" font="vector"/>
 <attribute name="VALUE" x="-53.34" y="269.24" size="1.27" layer="96" font="vector"/>
+</instance>
+<instance part="NEO_PIXEL" gate="-1" x="-99.06" y="220.98" smashed="yes">
+<attribute name="NAME" x="-99.06" y="221.869" size="1.778" layer="95" rot="R180"/>
+</instance>
+<instance part="NEO_PIXEL" gate="-2" x="-99.06" y="215.9" smashed="yes">
+<attribute name="VALUE" x="-101.6" y="212.217" size="1.778" layer="96"/>
+<attribute name="NAME" x="-99.06" y="216.789" size="1.778" layer="95" rot="R180"/>
 </instance>
 </instances>
@@
 <wire x1="-162.56" y1="220.98" x2="-170.18" y2="220.98" width="0.1524" layer="91"/>
 <label x="-172.72" y="220.98" size="0.8128" layer="95" rot="R180" xref="yes"/>
-</segment>
-<segment>
-<pinref part="NEO_PIXEL" gate="-3" pin="SK"/>
-<wire x1="-93.98" y1="215.9" x2="-81.28" y2="215.9" width="0.1524" layer="91"/>
-<label x="-81.28" y="218.44" size="1.778" layer="95" rot="R180"/>
-<label x="-78.74" y="215.9" size="0.8128" layer="95" xref="yes"/>
 </segment>
 <segment>
@@
 <label x="104.14" y="111.76" size="0.8128" layer="95" xref="yes"/>
 </segment>
+<segment>
+<pinref part="NEO_PIXEL" gate="-2" pin="KL"/>
+<wire x1="-93.98" y1="215.9" x2="-81.28" y2="215.9" width="0.1524" layer="91"/>
+<label x="-78.74" y="215.9" size="0.8128" layer="95" xref="yes"/>
+</segment>
 </net>
 <net name="5V" class="0">
@@
 <wire x1="124.46" y1="121.92" x2="109.22" y2="121.92" width="0.1524" layer="91"/>
 <label x="106.68" y="121.92" size="0.8128" layer="95" rot="R180" xref="yes"/>
-</segment>
-<segment>
-<pinref part="NEO_PIXEL" gate="-2" pin="SK"/>
-<wire x1="-93.98" y1="220.98" x2="-81.28" y2="220.98" width="0.1524" layer="91"/>
-<label x="-81.28" y="223.52" size="1.778" layer="95" rot="R180"/>
-<label x="-78.74" y="220.98" size="0.8128" layer="95" xref="yes"/>
 </segment>
 <segment>
@@
 </segment>
 <segment>
-<pinref part="NEO_PIXEL" gate="-1" pin="SK"/>
-<wire x1="-93.98" y1="226.06" x2="-81.28" y2="226.06" width="0.1524" layer="91"/>
-<label x="-81.28" y="228.6" size="1.778" layer="95" rot="R180"/>
-<label x="-78.74" y="226.06" size="0.8128" layer="95" xref="yes"/>
-</segment>
-</net>
+<pinref part="NEO_PIXEL" gate="-1" pin="KL"/>
+<wire x1="-93.98" y1="220.98" x2="-81.28" y2="220.98" width="0.1524" layer="91"/>
+<label x="-78.74" y="220.98" size="0.8128" layer="95" xref="yes"/>
+</segment>
+</net>
